File: stepomatic.kicad_pcb (KiCad board)
At the start: 2 copper layers, 50 x 30 mm, 43 parts, among them J1 I2C, J4 USB_B_Micro, Q1 MMBT3904, Q2 MMBT3904, SW1 Mode, SW2 RST, U1 HDC1080DMBR, U2 AMS1117-3.3, U3 ULN2003A, U4 CH340C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

Commit message: Tidy up for review
Changed lines of the file:
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@@
     (fp_line (start -0.295631 -0.715443) (end -1.095631 -0.715443) (layer "F.SilkS") (width 0.254001))
     (fp_arc (start -1.405512 -0.405613) (mid -1.314765 -0.624696) (end -1.095682 -0.715443) (layer "F.SilkS") (width 0.254001))
-    (fp_arc (start 1.390018 0.400203) (mid 1.299267 0.619284) (end 1.080188 0.710033) (layer "F.SilkS") (width 0.254001))
+    (fp_arc (start 1.390018 0.400203) (mid 1.299267 0.61928) (end 1.080188 0.710033) (layer "F.SilkS") (width 0.254001))
     (fp_arc (start -1.095682 0.704216) (mid -1.314773 0.61346) (end -1.405511 0.394362) (layer "F.SilkS") (width 0.254001))
     (fp_arc (start 1.080188 -0.709627) (mid 1.299286 -0.618875) (end 1.390018 -0.399772) (layer "F.SilkS") (width 0.254001))
@@
       (effects (font (size 1 1) (thickness 0.15)))
     )
-    (fp_text value "USB_B_Micro" (at 0.170278 4.688035 90) (layer "F.SilkS")
-      (effects (font (size 1 1) (thickness 0.15)))
-    )
+    (fp_text value "USB_B_Micro" (at 0.170278 4.688035 90) (layer "F.SilkS") hide
+      (effects (font (size 1 1) (thickness 0.15)))
+    )
